File: board/sonic-telemeter.brd (EAGLE design)
At the start: 100 x 80 mm, 31 parts, among them T1 2N2222, T2 2N2222

Commit message: Fix board
Parts:
- removed IC2, IC6: (no value), ic-package:DIL16
- moved JP1 78.3 mm to (96.5, 64.8), turned to 90 degrees
- moved IC1 61.1 mm to (73.7, 47.0), turned to 90 degrees
- moved R19 54.3 mm to (48.3, 14.0), turned to 180 degrees
- moved R16 51.7 mm to (39.4, 14.0), turned to 180 degrees
- moved T1 48.9 mm to (49.5, 19.1)
- moved T2 45.0 mm to (40.6, 19.1)
- moved R3 42.2 mm to (33.0, 48.3), turned to 0 degrees
- moved R4 40.1 mm to (33.0, 45.7), turned to 0 degrees
- moved R5 36.6 mm to (33.0, 40.6), turned to 0 degrees
- moved R8 35.2 mm to (33.0, 38.1), turned to 0 degrees
- moved R11 34.2 mm to (33.0, 35.6), turned to 0 degrees
- moved R12 33.5 mm to (33.0, 33.0), turned to 0 degrees
- moved R13 33.3 mm to (33.0, 27.9), turned to 0 degrees
- moved R1 26.2 mm to (58.4, 48.3), turned to 180 degrees
- moved DIS2 24.3 mm to (45.7, 43.2), turned to 270 degrees
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Connections:
- net N$1 renamed STRG
- net N$3 renamed SECH
- net N$40 renamed AL1
- net N$41 renamed AL2
- net N$44 renamed GND3
- net N$47 renamed GND2
- removed net N$10: IC2.13, R5.1
- removed net N$11: IC1.2, IC2.12, R4.1
- removed net N$19: IC1.15, R3.1
- removed net N$21: IC1.14, R2.1
- removed net N$22: IC2.2, IC6.12
- removed net N$24: IC1.13, R1.1
- removed net N$25: IC1.12, R8.1
- removed net N$26: IC5.14, R14.1
- removed net N$27: IC6.13, R9.1
- removed net N$36: R16.2, U$1.21
- removed net N$37: IC6.14, R10.1
- removed net N$38: T1.1, T2.1, U$1.23
- removed net N$39: R19.2, U$1.22
- removed net N$48: IC1.11, IC2.11, IC5.11, IC6.11, U$1.1
- removed net N$49: IC1.10, IC1.8, IC2.10, IC2.8, IC5.10, IC5.8, IC6.10, IC6.8, U$1.3
- removed net N$51: IC6.15, R11.1
- removed net N$9: IC2.14, R6.1
- new net DCK: IC1.9, IC5.9, U$1.19
- new net DDS: IC5.2, U$1.17
- new net DDW: IC1.11, IC5.11, U$1.20
- new net DEN1: R19.2, U$1.1
- new net DEN2: R16.2, U$1.2
- new net GND1: IC1.10, IC1.8, IC5.10, IC5.8, T1.1, T2.1, U$1.18
- new net N$1: IC1.15, R6.1, R8.1
- new net N$3: IC1.13, R2.1, R4.1
- net N$2: now also IC1.14, R5.1, R7.1; no longer IC5.2, U$1.4
- net N$4: now also IC1.12, R1.1, R3.1; no longer IC1.9, IC2.9, IC5.9, IC6.9, U$1.2
- net N$45: now also IC1.2, R11.1, R9.1; no longer IC6.2, R12.1
- net N$46: now also IC5.14, R13.1; no longer IC5.15
- net N$5: now also R10.1, R12.1; no longer R13.1
- net N$6: now also IC5.15, R14.1; no longer IC2.15, R7.1
- net VCC1: no longer IC2.1, IC2.16, IC6.1, IC6.16
Routing:
- net N$11: track 163.0 -> 0.00 mm
- net GND1: track 0.00 -> 138.0 mm
- net N$49: track 126.6 -> 0.00 mm
- net N$48: track 122.8 -> 0.00 mm
- net N$8: track 142.3 -> 29.3 mm
- net N$7: track 173.7 -> 62.2 mm
- net N$4: track 146.2 -> 40.5 mm
- net N$19: track 89.2 -> 0.00 mm
- net DDS: track 0.00 -> 83.3 mm
- net STRG: track 3.51 -> 81.4 mm
- net GND2: track 4.48 -> 81.9 mm
- net N$25: track 73.4 -> 0.00 mm
- net DEN1: track 0.00 -> 71.3 mm
- net SECH: track 8.41 -> 75.3 mm
- net VCC1: track 304.4 -> 243.4 mm
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